Commit message: finished milestone 2

File: body.urdf (robot description, URDF)
Before this commit: robot robot, 9 links, 8 joints
Links:
- removed link BackLeg
- removed link BackLowerLeg
- removed link FrontLeg
- removed link FrontLowerLeg
- removed link LeftLeg
- removed link RightLeg
- added link LeftFoot, mass 1; collision box size=1 1.5 0.5; visual box size=1 1.5 0.5
- added link LeftLowerArm, mass 1; collision box size=1 1 2; visual box size=1 1 2
- added link LeftUpperArm, mass 1; collision box size=1 1 2; visual box size=1 1 2
- added link LeftUpperLeg, mass 1; collision box size=1 1 2; visual box size=1 1 2
- added link RightFoot, mass 1; collision box size=1 1.5 0.5; visual box size=1 1.5 0.5
- added link RightLowerArm, mass 1; collision box size=1 1 2; visual box size=1 1 2
- added link RightUpperArm, mass 1; collision box size=1 1 2; visual box size=1 1 2
- added link RightUpperLeg, mass 1; collision box size=1 1 2; visual box size=1 1 2
- link LeftLowerLeg: geometry collision box size=1 1 2; visual box size=1 1 2
- link RightLowerLeg: geometry collision box size=1 1 2; visual box size=1 1 2
- link Torso: geometry collision box size=2 1 4; visual box size=2 1 4
Joints:
- removed joint BackLeg_BackLowerLeg
- removed joint FrontLeg_FrontLowerLeg
- removed joint LeftLeg_LeftLowerLeg
- removed joint RightLeg_RightLowerLeg
- removed joint Torso_BackLeg
- removed joint Torso_FrontLeg
- removed joint Torso_LeftLeg
- removed joint Torso_RightLeg
- added joint LeftLowerLeg_LeftFoot: type revolute, parent LeftLowerLeg, child LeftFoot, origin xyz=0 0 -2 rpy=0 0 0, axis 1 0 0, limit lower=-3.14159 upper=3.14159 effort=0.0 velocity=0.0
- added joint LeftUpperArm_LeftLowerArm: type revolute, parent LeftUpperArm, child LeftLowerArm, origin xyz=0.5 0 -1.5 rpy=0 0 0, axis 1 0 0, limit lower=-3.14159 upper=3.14159 effort=0.0 velocity=0.0
- added joint LeftUpperLeg_LeftLowerLeg: type revolute, parent LeftUpperLeg, child LeftLowerLeg, origin xyz=0 0 -2 rpy=0 0 0, axis 1 0 0, limit lower=-3.14159 upper=3.14159 effort=0.0 velocity=0.0
- added joint RightLowerLeg_RightFoot: type revolute, parent RightLowerLeg, child RightFoot, origin xyz=0 0 -2 rpy=0 0 0, axis 1 0 0, limit lower=-3.14159 upper=3.14159 effort=0.0 velocity=0.0
- added joint RightUpperArm_RightLowerArm: type revolute, parent RightUpperArm, child RightLowerArm, origin xyz=-0.5 0 -1.5 rpy=0 0 0, axis 1 0 0, limit lower=-3.14159 upper=3.14159 effort=0.0 velocity=0.0
- added joint RightUpperLeg_RightLowerLeg: type revolute, parent RightUpperLeg, child RightLowerLeg, origin xyz=0 0 -2 rpy=0 0 0, axis 1 0 0, limit lower=-3.14159 upper=3.14159 effort=0.0 velocity=0.0
- added joint Torso_LeftUpperArm: type revolute, parent Torso, child LeftUpperArm, origin xyz=1 0 8 rpy=0 0 0, axis 1 0 0, limit lower=-3.14159 upper=3.14159 effort=0.0 velocity=0.0
- added joint Torso_LeftUpperLeg: type revolute, parent Torso, child LeftUpperLeg, origin xyz=0.75 0 4.5 rpy=0 0 0, axis 1 0 0, limit lower=-3.14159 upper=3.14159 effort=0.0 velocity=0.0
- added joint Torso_RighUpperArm: type revolute, parent Torso, child RightUpperArm, origin xyz=-1 0 8 rpy=0 0 0, axis 1 0 0, limit lower=-3.14159 upper=3.14159 effort=0.0 velocity=0.0
- added joint Torso_RightUpperLeg: type revolute, parent Torso, child RightUpperLeg, origin xyz=-0.75 0 4.5 rpy=0 0 0, axis 1 0 0, limit lower=-3.14159 upper=3.14159 effort=0.0 velocity=0.0

Commit message: finished milestone 3

File: body.urdf (robot description, URDF)
Before this commit: robot robot, 11 links, 10 joints
Joints:
- removed joint Torso_RighUpperArm
- added joint Torso_RightUpperArm: type revolute, parent Torso, child RightUpperArm, origin xyz=-1 0 8 rpy=0 0 0, axis 1 0 0, limit lower=-3.14159 upper=3.14159 effort=0.0 velocity=0.0
